File: picsy-hw/picsy-hw.kicad_pcb (KiCad board)
At the start: 2 copper layers, 125 x 55 mm, 112 parts, among them J1 Power/Data, J2 BATT, J3 Cam, J5 SD, J6 0.99" Display, J7 2" Display, P2 TC2030-CTX-Tag-Connect, Q1 S8050, Q2 S8050, Q3 AO3401A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

Commit message: updated hw files
Parts:
- added REF**: DISPLAY-0.99", otter:DUMMY-3D, F.Cu at (133.0, 100.8)
- added REF**: DISPLAY-2.0", otter:DUMMY-3D, F.Cu at (61.8, 87.5)
