File: picsy-hw/picsy-hw.kicad_sch (KiCad schematic)
At the start: 112 parts, among them J1 Power/Data, J2 BATT, J3 Cam, J4 Cam, J5 SD, J6 0.99" Display, J7 2" Display, P2 TC2030-CTX-Tag-Connect, Q1 S8050, Q2 S8050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

Commit message: updated hw files
Parts:
- C22: value 100n -> 15p
- R18, R22: value 47k -> DNP
Connections:
- net ESP_RX: now also U1.2 (TXD); no longer U1.3 (RXD)
- net ESP_TX: now also U1.3 (RXD); no longer U1.2 (TXD)
- net PSRAM_SD2: now also U6.7 (SIO3); no longer U6.3 (SIO2)
- net PSRAM_SD3: now also U6.3 (SIO2); no longer U6.7 (SIO3)
Other:
- note added: "VERSION 2: - fix psram pinout - swap sub-nibbles for pin 2 and 3 [DONE] - Cam-Clock pin to 15pf [DONE] - Font size too small - Status LEDs - Back and Front - Display Backlight - STM32 I2C Bootloader - SD CARD Single lane interface? - ESP32 to ESP32-Mini or other modern Module - FIX UART [DONE]"
- note removed: "TODO: - Double Check - Status LEDs"
Changed lines of the file:
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@@
 		)
 	)
-	(text "TODO:\n - Double Check\n - Status LEDs"
+	(text "VERSION 2:\n - fix psram pinout\n    - swap sub-nibbles for pin 2 and 3 [DONE]\n - Cam-Clock pin to 15pf [DONE]\n - Font size too small\n - Status LEDs\n	- Back and Front\n - Display Backlight\n - STM32 I2C Bootloader\n - SD CARD Single lane interface?\n - ESP32 to ESP32-Mini or other modern Module\n - FIX UART [DONE]"
 		(exclude_from_sim no)
 		(at 102.108 80.518 0)
@@
 	(global_label "ESP_RX"
 		(shape input)
-		(at 82.55 -35.56 0)
+		(at 82.55 -38.1 0)
 		(fields_autoplaced yes)
 		(effects
@@
 		)
 		(property "Intersheetrefs" "${INTERSHEET_REFS}"
-			(at -24.13 -62.23 0)
+			(at 92.6108 -38.1 0)
 			(effects
 				(font
 					(size 1.27 1.27)
 				)
+				(justify left)
 				(hide yes)
 			)
@@
 	(global_label "PSRAM_SD3"
 		(shape input)
-		(at 199.39 91.44 180)
+		(at 199.39 93.98 180)
 		(fields_autoplaced yes)
 		(effects
@@
 		)
 		(property "Intersheetrefs" "${INTERSHEET_REFS}"
-			(at 185.4587 91.44 0)
+			(at 185.4587 93.98 0)
 			(effects
 				(font
@@
 	(global_label "PSRAM_SD2"
 		(shape input)
-		(at 199.39 93.98 180)
+		(at 199.39 91.44 180)
 		(fields_autoplaced yes)
 		(effects
@@
 		)
 		(property "Intersheetrefs" "${INTERSHEET_REFS}"
-			(at 185.4587 93.98 0)
+			(at 185.4587 91.44 0)
 			(effects
 				(font
@@
 	(global_label "ESP_TX"
 		(shape input)
-		(at 82.55 -38.1 0)
+		(at 82.55 -35.56 0)
 		(fields_autoplaced yes)
 		(effects
@@
 		)
 		(property "Intersheetrefs" "${INTERSHEET_REFS}"
-			(at 92.3084 -38.1 0)
+			(at 92.3084 -35.56 0)
 			(effects
 				(font
@@
 			)
 		)
-		(property "Value" "47k"
+		(property "Value" "DNP"
 			(at 218.44 129.54 90)
 			(effects
@@
 			)
 		)
-		(property "Value" "47k"
+		(property "Value" "DNP"
 			(at 218.44 144.78 90)
 			(effects
@@
 			)
 		)
-		(property "Value" "100n"
+		(property "Value" "15p"
 			(at 152.4 104.1462 0)
 			(effects

Commit message: updated schematic
Other:
- note added: "VERSION 2: - fix psram pinout [DONE] - swap sub-nibbles for pin 2 and 3 [DONE] - Cam-Clock pin to 15pf [DONE] - Font size too small - Status LEDs - Back and Front - Display Backlight - STM32 I2C Bootloader - SD CARD Single lane interface? - ESP32 to ESP32-Mini or other modern Module - FIX UART [DONE]"
- note removed: "VERSION 2: - fix psram pinout - swap sub-nibbles for pin 2 and 3 [DONE] - Cam-Clock pin to 15pf [DONE] - Font size too small - Status LEDs - Back and Front - Display Backlight - STM32 I2C Bootloader - SD CARD Single lane interface? - ESP32 to ESP32-Mini or other modern Module - FIX UART [DONE]"
Changed lines of the file:
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@@
 		)
 	)
-	(text "VERSION 2:\n - fix psram pinout\n    - swap sub-nibbles for pin 2 and 3 [DONE]\n - Cam-Clock pin to 15pf [DONE]\n - Font size too small\n - Status LEDs\n	- Back and Front\n - Display Backlight\n - STM32 I2C Bootloader\n - SD CARD Single lane interface?\n - ESP32 to ESP32-Mini or other modern Module\n - FIX UART [DONE]"
+	(text "VERSION 2:\n - fix psram pinout [DONE]\n    - swap sub-nibbles for pin 2 and 3 [DONE]\n - Cam-Clock pin to 15pf [DONE]\n - Font size too small\n - Status LEDs\n	- Back and Front\n - Display Backlight\n - STM32 I2C Bootloader\n - SD CARD Single lane interface?\n - ESP32 to ESP32-Mini or other modern Module\n - FIX UART [DONE]"
 		(exclude_from_sim no)
 		(at 102.108 80.518 0)

Commit message: updated schematic todo
Connections:
- net Brightness renamed Exposure
- net Resolution renamed Dither
Other:
- note added: "VERSION 2: - fix psram pinout [DONE] - swap sub-nibbles for pin 2 and 3 [DONE] - Cam-Clock pin to 15pf [DONE] - Font size too small - Status LEDs - Back and Front - Display Backlight - STM32 I2C Bootloader - SD CARD Single lane interface? - ESP32 to ESP32-Mini or other modern Module - FIX UART [DONE] - STM32 nRST PullUp - Live view display connector too narrow"
- note removed: "VERSION 2: - fix psram pinout [DONE] - swap sub-nibbles for pin 2 and 3 [DONE] - Cam-Clock pin to 15pf [DONE] - Font size too small - Status LEDs - Back and Front - Display Backlight - STM32 I2C Bootloader - SD CARD Single lane interface? - ESP32 to ESP32-Mini or other modern Module - FIX UART [DONE]"
Changed lines of the file:
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@@
 		)
 	)
-	(text "VERSION 2:\n - fix psram pinout [DONE]\n    - swap sub-nibbles for pin 2 and 3 [DONE]\n - Cam-Clock pin to 15pf [DONE]\n - Font size too small\n - Status LEDs\n	- Back and Front\n - Display Backlight\n - STM32 I2C Bootloader\n - SD CARD Single lane interface?\n - ESP32 to ESP32-Mini or other modern Module\n - FIX UART [DONE]"
+	(text "VERSION 2:\n - fix psram pinout [DONE]\n    - swap sub-nibbles for pin 2 and 3 [DONE]\n - Cam-Clock pin to 15pf [DONE]\n - Font size too small\n - Status LEDs\n	- Back and Front\n - Display Backlight\n - STM32 I2C Bootloader\n - SD CARD Single lane interface?\n - ESP32 to ESP32-Mini or other modern Module\n - FIX UART [DONE]\n - STM32 nRST PullUp\n - Live view display connector too narrow"
 		(exclude_from_sim no)
 		(at 102.108 80.518 0)
@@
 		)
 	)
-	(global_label "Brightness"
+	(global_label "Exposure"
 		(shape input)
 		(at 76.2 295.91 180)
@@
 		)
 		(property "Intersheetrefs" "${INTERSHEET_REFS}"
-			(at 63.2363 295.91 0)
+			(at 64.6878 295.91 0)
 			(effects
 				(font
@@
 		)
 	)
-	(global_label "Resolution"
+	(global_label "Dither"
 		(shape input)
 		(at 22.86 257.81 0)
@@
 		)
 		(property "Intersheetrefs" "${INTERSHEET_REFS}"
-			(at 35.8236 257.81 0)
+			(at 31.4695 257.81 0)
 			(effects
 				(font
@@
 		)
 	)
-	(global_label "Resolution"
+	(global_label "Dither"
 		(shape input)
 		(at 76.2 224.79 180)
@@
 		)
 		(property "Intersheetrefs" "${INTERSHEET_REFS}"
-			(at 63.2364 224.79 0)
+			(at 67.5905 224.79 0)
 			(effects
 				(font
@@
 		)
 	)
-	(global_label "Brightness"
+	(global_label "Exposure"
 		(shape input)
 		(at 22.86 262.89 0)
@@
 		)
 		(property "Intersheetrefs" "${INTERSHEET_REFS}"
-			(at 35.8237 262.89 0)
-			(effects
-				(font
+			(at 34.3722 262.89 0)
+			(effects
+				(font
